Commit message: added tuto source, changed Red/Blue colors to grey, param loaded directly at startup

File: mybot_description/urdf/mybot.xacro (robot description, xacro)
@@ -58,5 +58,4 @@
 	<sphere radius="${casterRadius}"/>
       </geometry>
-      <material name="red"/>
     </visual>
     <inertial>
